Commit message: add realsense d435i to URDF

File: robot_sd700e_description/urdf/robot_sd700e.xacro (robot description, xacro)
@@ -50,4 +50,5 @@
     <parent link="base_link" />
     <child link="link1" />
+    <!--axis xyz="0 0 -1" /-->
     <axis xyz="0 0 1" />
     <limit lower="-2.96" upper="2.96" effort="100" velocity="1" />
@@ -78,7 +79,9 @@
   <joint name="joint2" type="revolute">
     <origin xyz="0 0 0.118" rpy="1.5708 -1.5708 3.1416" />
+    <!--origin xyz="0 0 0.118" rpy="${M_PI / 2} 0 0" / -->
     <parent link="link1" />
     <child link="link2" />
-    <axis xyz="0 0 -1" />
+    <axis xyz="0 0 1" />
+    <!--axis xyz="0 0 -1" /-->
     <limit lower="-1.91" upper="1.91" effort="100" velocity="1" />
   </joint>
@@ -138,5 +141,6 @@
     <parent link="link3" />
     <child link="link4" />
-    <axis xyz="0 0 -1" />
+    <!--axis xyz="0 0 -1" /-->
+    <axis xyz="0 0 1" />
     <limit lower="-3.22" upper="3.22" effort="100" velocity="1" />
   </joint>
@@ -196,4 +200,5 @@
     <parent link="link5" />
     <child link="link6" />
+    <!--axis xyz="0 0 -1" /-->
     <axis xyz="0 0 1" />
     <limit lower="-6.28" upper="6.28" effort="100" velocity="1" />

Commit message: update

File: robot_sd700e_description/urdf/robot_sd700e.xacro (robot description, xacro)
@@ -5,6 +5,8 @@
     <inertial>
       <origin xyz="-0.0194690222590369 -0.000269188119329771 0.0669003838868867" rpy="0 0 0" />
-      <mass value="0.00001" />
+      <!--<mass value="0.00001" />-->
+      <mass value="0.1" />
       <inertia ixx="0.000153169404327002" ixy="1.65882461270346E-10" ixz="4.4079170251983E-07" iyy="0.000178370863576969" iyz="-2.76318351033745E-09" izz="0.000146674461881756" />
+      <!--<inertia ixx="0" ixy="0" ixz="0" iyy="0" iyz="0" izz="0" /> -->
     </inertial>
     <visual>
@@ -29,4 +31,5 @@
       <mass value="0.00001" />
       <inertia ixx="4.83982220972564E-05" ixy="-1.77040002978859E-10" ixz="3.19080107721578E-11" iyy="4.76414174481088E-05" iyz="-1.87834825511904E-09" izz="3.52854220263338E-05" />
+      <!--<inertia ixx="0" ixy="0" ixz="0" iyy="0" iyz="0" izz="0" />-->
     </inertial>
     <visual>
@@ -178,5 +181,5 @@
       <origin xyz="2.98155597433514E-18 -2.16840434497101E-17 0.013" rpy="0 0 0" />
       <mass value="0.00001" />
-      <inertia ixx="5.12858666666666E-06" ixy="1.96434522866803E-23" ixz="1.31858481743306E-22" iyy="3.04650666666666E-06" iyz="-4.7358312294891E-23" izz="5.12858666666666E-06" />
+      <inertia ixx="0" ixy="0" ixz="0" iyy="0" iyz="0" izz="0" />
     </inertial>
     <visual>
