Commit message: update

File: robot_sd700e_description/urdf/robot_sd700e_with_kinect.xacro (robot description, xacro)
@@ -14,6 +14,13 @@
   </joint>
 -->
+  <!-- kinect parent = link7 -->
+  <!--
   <sensor_d435 parent="link7">
     <origin xyz="${kinect_offset_x} ${kinect_offset_y} ${kinect_offset_z}" rpy="0 -1.5707 3.14159"/>
   </sensor_d435>
+  -->
+  <!-- kinect parent = base_link -->
+  <sensor_d435 parent="base_link">
+    <origin xyz="0.7 0 0.7" rpy="0 1.5707 0"/>
+  </sensor_d435>
 </robot>

Commit message: update

File: robot_sd700e_description/urdf/robot_sd700e_with_kinect.xacro (robot description, xacro)
@@ -3,7 +3,10 @@
   <xacro:include filename="$(find robot_sd700e_description)/urdf/robot_sd700e.xacro" />
   <xacro:include filename="$(find realsense2_description)/urdf/_d435.urdf.xacro" />
-  <xacro:property name="kinect_offset_x" value="0.05" />
-  <xacro:property name="kinect_offset_y" value="0" />
-  <xacro:property name="kinect_offset_z" value="0" />
+  <xacro:property name="kinect_offset_x" value="0.647" />
+  <xacro:property name="kinect_offset_y" value="0.955" />
+  <xacro:property name="kinect_offset_z" value="0.689" />
+  <xacro:property name="kinect_RPY_x" value="-3.08076" />
+  <xacro:property name="kinect_RPY_y" value="-0.0440471" />
+  <xacro:property name="kinect_RPY_z" value="-2.04154" />
   <!-- Kinect -->
   <!--
@@ -22,5 +25,5 @@
   <!-- kinect parent = base_link -->
   <sensor_d435 parent="base_link">
-    <origin xyz="0.7 0 0.7" rpy="0 1.5707 0"/>
+    <origin xyz="${kinect_offset_x} ${kinect_offset_y} ${kinect_offset_z}" rpy="${kinect_RPY_x} ${kinect_offset_y} ${kinect_RPY_z}"/>
   </sensor_d435>
 </robot>

Commit message: update

File: robot_sd700e_description/urdf/robot_sd700e_with_kinect.xacro (robot description, xacro)
@@ -3,17 +3,26 @@
   <xacro:include filename="$(find robot_sd700e_description)/urdf/robot_sd700e.xacro" />
   <xacro:include filename="$(find realsense2_description)/urdf/_d435.urdf.xacro" />
-  <xacro:property name="kinect_offset_x" value="0.647" />
-  <xacro:property name="kinect_offset_y" value="0.955" />
-  <xacro:property name="kinect_offset_z" value="0.689" />
-  <xacro:property name="kinect_RPY_x" value="-3.08076" />
-  <xacro:property name="kinect_RPY_y" value="-0.0440471" />
-  <xacro:property name="kinect_RPY_z" value="-2.04154" />
-  <!-- Kinect -->
-  <!--
-  <joint name="kinect_joint" type="fixed">
-    <origin xyz="${kinect_offset_x} ${kinect_offset_y} ${kinect_offset_z}" rpy="0 1.5707 1.570" />
-    <parent link="base_link"/>
-    <child link="sensor_d435_link"/>
-  </joint>
+<!--
+  <xacro:property name="kinect_offset_x" value="0.620" />
+  <xacro:property name="kinect_offset_y" value=" 0.959" />
+  <xacro:property name="kinect_offset_z" value="0.645" />
+  <xacro:property name="kinect_RPY_x" value="-0.047" />
+  <xacro:property name="kinect_RPY_y" value="0.471" />
+  <xacro:property name="kinect_RPY_z" value="-1.665" />
+-->
+  <!-- latest 2020-01-08 -->
+  <xacro:property name="kinect_offset_x" value="0.618" />
+  <xacro:property name="kinect_offset_y" value=" 0.975" />
+  <xacro:property name="kinect_offset_z" value="0.661" />
+  <xacro:property name="kinect_RPY_x" value="-0.067" />
+  <xacro:property name="kinect_RPY_y" value=" 0.487" />
+  <xacro:property name="kinect_RPY_z" value="-1.638" />
+<!--
+  <xacro:property name="kinect_offset_x" value="0.618" />
+  <xacro:property name="kinect_offset_y" value=" 0.975" />
+  <xacro:property name="kinect_offset_z" value="0.661" />
+  <xacro:property name="kinect_RPY_x" value="0.00" />
+  <xacro:property name="kinect_RPY_y" value="0.00" />
+  <xacro:property name="kinect_RPY_z" value="0.00" />
 -->
   <!-- kinect parent = link7 -->
@@ -25,5 +34,5 @@
   <!-- kinect parent = base_link -->
   <sensor_d435 parent="base_link">
-    <origin xyz="${kinect_offset_x} ${kinect_offset_y} ${kinect_offset_z}" rpy="${kinect_RPY_x} ${kinect_offset_y} ${kinect_RPY_z}"/>
-  </sensor_d435>
+    <origin xyz="${kinect_offset_x} ${kinect_offset_y} ${kinect_offset_z}" rpy="${kinect_RPY_x} ${kinect_RPY_y} ${kinect_RPY_z}"/>
+  </sensor_d435>                 2
 </robot>

Commit message: update

File: robot_sd700e_description/urdf/robot_sd700e_with_kinect.xacro (robot description, xacro)
@@ -18,12 +18,4 @@
   <xacro:property name="kinect_RPY_y" value=" 0.487" />
   <xacro:property name="kinect_RPY_z" value="-1.638" />
-<!--
-  <xacro:property name="kinect_offset_x" value="0.618" />
-  <xacro:property name="kinect_offset_y" value=" 0.975" />
-  <xacro:property name="kinect_offset_z" value="0.661" />
-  <xacro:property name="kinect_RPY_x" value="0.00" />
-  <xacro:property name="kinect_RPY_y" value="0.00" />
-  <xacro:property name="kinect_RPY_z" value="0.00" />
--->
   <!-- kinect parent = link7 -->
   <!--

Commit message: update relationship between robot and camera

File: robot_sd700e_description/urdf/robot_sd700e_with_kinect.xacro (robot description, xacro)
@@ -12,4 +12,5 @@
 -->
   <!-- latest 2020-01-08 -->
+<!--
   <xacro:property name="kinect_offset_x" value="0.618" />
   <xacro:property name="kinect_offset_y" value=" 0.975" />
@@ -18,4 +19,12 @@
   <xacro:property name="kinect_RPY_y" value=" 0.487" />
   <xacro:property name="kinect_RPY_z" value="-1.638" />
+-->
+  <!-- latest 2020-01-14 -->
+  <xacro:property name="kinect_offset_x" value="0.622" />
+  <xacro:property name="kinect_offset_y" value=" 0.968" />
+  <xacro:property name="kinect_offset_z" value="0.641" />
+  <xacro:property name="kinect_RPY_x" value="-0.062" />
+  <xacro:property name="kinect_RPY_y" value=" 0.467" />
+  <xacro:property name="kinect_RPY_z" value="-1.637" />
   <!-- kinect parent = link7 -->
   <!--
@@ -27,4 +36,4 @@
   <sensor_d435 parent="base_link">
     <origin xyz="${kinect_offset_x} ${kinect_offset_y} ${kinect_offset_z}" rpy="${kinect_RPY_x} ${kinect_RPY_y} ${kinect_RPY_z}"/>
-  </sensor_d435>                 2
+  </sensor_d435>
 </robot>
